File: Hardware/Eagle/CompleteGameBoard/CompleteBoard.brd (EAGLE design)
At the start: 6.2 x 4.2 mm, 21 parts

Commit message: Updated Wiring and parts for issue #12 so that through hole buttons are used
Parts:
- S0, S1, S2, S3, S4: value MOMENTARY-SWITCH-SPST-SMD-12MM -> MOMENTARY-SWITCH-SPST-PTH-12MM; device SparkFun-Switches:TACTILE_SWITCH_SMD_12MM -> SparkFun-Switches:TACTILE_SWITCH_PTH_12MM
- moved R5 256.1 mm to (143.5, 52.1)
- moved R6 235.4 mm to (109.2, 49.5)
- moved D1 222.7 mm to (137.2, 45.7)
- moved S5 222.3 mm to (124.5, 45.7)
- moved LS2 216.6 mm to (73.7, 52.1)
- moved D2 211.2 mm to (113.0, 45.7)
- moved LS1 210.9 mm to (7.62, 52.1)
- moved A3 173.3 mm to (95.2, 35.6), turned to 270 degrees
- moved R1 144.4 mm to (-71.1, -95.2)
- moved R0 144.4 mm to (-78.7, -95.2)
- moved S2 136.3 mm to (-91.4, -85.1)
- moved S3 136.3 mm to (-73.7, -85.1)
- moved A2 114.5 mm to (-99.1, -61.0)
- moved S0 114.5 mm to (-91.4, -69.8)
- moved S1 114.5 mm to (-73.7, -69.8)
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Connections:
- net 3.3V: now also S1.4; no longer S1.3, S4.3
- net BUTTON0: now also S0.2; no longer S0.1
- net BUTTON4: now also A1.9@J4; no longer R4.2, S4.1
- net GND: no longer R4.1
Other:
- board size 6.2 x 4.2 mm -> 149.9 x 97.8 mm
