File: Hardware/Eagle/GameControllerBoard/ControllerBoard.brd (EAGLE design)
At the start: 6.2 x 4.2 mm, 4 parts

Commit message: Added reference for button 4 for issue #7
Connections:
- net BUTTON4: now also A1.9@J4
Changed lines of the file:
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@@
 <signal name="BUTTON4">
 <contactref element="J2" pad="7"/>
+<contactref element="A1" pad="9@J4"/>
+<wire x1="11.43" y1="-46.99" x2="5.08" y2="-88.773" width="0" layer="19" extent="1-1"/>
 </signal>
 </signals>
