File: Hardware/Eagle/GameInterfaceBoard/InterfaceBoard.brd (EAGLE design)
At the start: 22 parts

Commit message: Added connection for button 4 and updated buttons to use through hole version and switched pins for easier connection on issue #2
Parts:
- removed A1: (no value), SparkFunBreakouts:LCD-15143
- removed U$1: COM-15168, SparkFunBreakouts:COM-15168
- added A2: TFT, SparkFunBreakouts:LCD-15143
- added A3: COM-15168, SparkFunBreakouts:COM-15168
- S0, S1, S2, S3, S4: value MOMENTARY-SWITCH-SPST-SMD-12MM -> MOMENTARY-SWITCH-SPST-PTH-12MM; device SparkFun-Switches:TACTILE_SWITCH_SMD_12MM -> SparkFun-Switches:TACTILE_SWITCH_PTH_12MM
- S5: value (none) -> STANDBY
- moved R6 186.0 mm to (-166.4, -27.9)
- moved R5 175.5 mm to (-160.0, -17.8)
- moved D2 175.3 mm to (-166.4, -20.3)
- moved S5 167.1 mm to (-166.4, -8.89)
- moved D1 165.9 mm to (-158.8, -6.35)
- moved J2 161.8 mm to (-167.6, -151.1)
- moved LS1 156.6 mm to (-137.2, -100.3)
- moved LS2 156.6 mm to (-124.5, -100.3)
- moved R4 133.5 mm to (69.8, 39.4), turned to 270 degrees
- moved R3 131.8 mm to (49.5, 44.5), turned to 180 degrees
- moved S4 103.4 mm to (67.3, 24.2), turned to 90 degrees
- moved R2 92.1 mm to (49.5, 27.9), turned to 180 degrees
- moved R0 91.5 mm to (49.5, 21.6), turned to 180 degrees
- moved R1 82.5 mm to (49.5, 15.2), turned to 180 degrees
- moved S3 74.3 mm to (23.2, 38.2), turned to 90 degrees
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Connections:
- removed net BUTTON5: R4.2, S4.1
- net 3.3V: now also A2.2@J2, S1.4, S4.4; no longer A1.2@J2, S1.3, S4.3
- net BUTTON0: now also S0.2; no longer S0.1
- net BUTTON4: now also R4.2, S4.1
- net CIPO: now also A2.6@J2; no longer A1.6@J2
- net COPI: now also A2.5@J2; no longer A1.5@J2
- net DC: now also A2.8@J2; no longer A1.8@J2
- net GND: now also A2.1@J2; no longer A1.1@J2
- net LCDCS: now also A2.9@J2; no longer A1.9@J2
- net PWM: now also A2.3@J2; no longer A1.3@J2
- net SCLK: now also A2.4@J2; no longer A1.4@J2
- net SDCS: now also A2.10@J2; no longer A1.10@J2
- net TE: now also A2.7@J2; no longer A1.7@J2
Routing:
- net 3.3V: track 0.00 -> 145.3 mm
- net GND: track 0.00 -> 49.5 mm
- net BUTTON2: track 0.00 -> 37.7 mm
- net BUTTON1: track 0.00 -> 21.4 mm
- net BUTTON3: track 0.00 -> 21.3 mm
- net BUTTON0: track 0.00 -> 9.05 mm
- net BUTTON4: track 0.00 -> 6.36 mm
Other:
- board outline added: 127 x 80 mm
