File: Hardware/KiCad/CompleteGameBoard/CompleteBoard.kicad_pcb (KiCad board)
At the start: 2 copper layers, 4.2 x 6.2 mm, 21 parts

Commit message: Re-imported updated EagleCAD board for issue #12
Parts:
- S0, S1, S2, S3, S4: value MOMENTARY-SWITCH-SPST-SMD-12MM -> MOMENTARY-SWITCH-SPST-PTH-12MM; footprint CompleteBoard:TACTILE_SWITCH_SMD_12MM -> CompleteBoard:TACTILE_SWITCH_PTH_12MM
- moved A2 138.8 mm to (93.9, 109.2), turned to 0 degrees
- moved R5 128.7 mm to (336.4, -3.86)
- moved A3 127.4 mm to (288.2, 12.6)
- moved D2 118.1 mm to (306.0, 2.49), turned to 0 degrees
- moved D1 117.0 mm to (330.1, 2.49), turned to 0 degrees
- moved R3 115.4 mm to (104.0, 158.7), turned to 0 degrees
- moved R6 115.3 mm to (302.2, -1.32), turned to 0 degrees
- moved S5 111.3 mm to (317.4, 2.49), turned to 0 degrees
- moved LS1 109.5 mm to (200.6, -3.86)
- moved R2 93.5 mm to (96.4, 158.7), turned to 0 degrees
- moved S3 91.7 mm to (119.3, 133.3), turned to 0 degrees
- moved LS2 90.3 mm to (266.6, -3.86)
- moved A1 83.8 mm to (137.1, 107.9), turned to 0 degrees
- moved R4 75.1 mm to (111.7, 158.7)
- moved R0 73.8 mm to (114.2, 143.5), turned to 0 degrees
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Connections:
- A1 pad 9@J4: Net-(A1-Pad9@J4) -> /BUTTON4
- R4 pad 1: GND -> Net-(R4-Pad1)
- R4 pad 2: /BUTTON4 -> Net-(R4-Pad2)
- S0 pad 1: /BUTTON0 -> Net-(S0-Pad1)
- S0 pad 2: (no net) -> /BUTTON0
- S0 pad 4: (no net) -> Net-(S0-Pad4)
- S1 pad 2: (no net) -> Net-(S1-Pad2)
- S1 pad 3: 3.3V -> Net-(S1-Pad3)
- S1 pad 4: (no net) -> 3.3V
- S2 pad 2: (no net) -> Net-(S2-Pad2)
- S2 pad 4: (no net) -> Net-(S2-Pad4)
- S3 pad 2: (no net) -> Net-(S3-Pad2)
- S3 pad 4: (no net) -> Net-(S3-Pad4)
- S4 pad 1: /BUTTON4 -> Net-(S4-Pad1)
- S4 pad 2: (no net) -> Net-(S4-Pad2)
- S4 pad 3: 3.3V -> Net-(S4-Pad3)
- S4 pad 4: (no net) -> Net-(S4-Pad4)
Routing:
- net /BUTTON3: track 7.01 -> 0.00 mm
- net /BUTTON2: track 5.85 -> 0.00 mm
Other:
- board size 4.2 x 6.2 mm -> 6.2 x 4.2 mm
